File: KiCad/ESP32_S3_PCB_TEMPLATE.kicad_sch (KiCad schematic)
At the start: 87 parts, among them CN3065_C2 4.7uF, CN3065_R1 1K8, CN3065_STDBY_LED1 LED, CN3965_C1 22uF, J1 Conn_01x07_Socket, J1 TYPE-C-31-M-12, J3 U.FL-R-SMT(01), J6 RFShield_OnePiece, U1 ATSHA204A-MAHDA-T, U1 MCP1525-TT, U3 Battery_charger_CN3065_QFN8, U4 AHT20, U6 TEMT6000

Commit message: Add files via upload
Parts:
- removed AUC1, VOLTAGE_REF_C1, VOLTAGE_REF_C2: 100nF, Capacitor_SMD:C_0603_1608Metric, symbol Device:C
- removed AUR1: AUR9718x_DFN_3x3mm_6_pin, Package_DFN_QFN:AUR9718 ST1S09 SON95P300X300X100-7N, symbol Power_Management:ST01S09_AUR9718x_DFN_3x3mm_6_pin
- removed AUR_C1: 22uF, Capacitor_SMD:C_0805_2012Metric_Pad1.18x1.45mm_HandSolder, symbol Device:C
- removed AUR_C2: 4.7uF, Capacitor_SMD:C_0805_2012Metric_Pad1.18x1.45mm_HandSolder, symbol Device:C
- removed AUR_R1: 75k, Resistor_SMD:R_0805_2012Metric_Pad1.20x1.40mm_HandSolder, symbol Device:R
- removed AUR_R2: 24k, Resistor_SMD:R_0805_2012Metric_Pad1.20x1.40mm_HandSolder, symbol Device:R
- removed AUR_l1: 3.3uF, Inductor_SMD:L_1210_3225Metric, symbol Device:L
- removed BAT_FUSE1, PWR_FUSE1: Polyfuse, Fuse:Fuse_1206_3216Metric_Pad1.42x1.75mm_HandSolder, symbol Device:Polyfuse
- removed BAT_SENSE_R1, BAT_SENSE_R2: 100k, Resistor_SMD:R_0603_1608Metric, symbol Device:R
- removed CN3065_C2: 4.7uF, Capacitor_SMD:C_0805_2012Metric, symbol Device:C
- removed CN3065_R1: 1K8, Resistor_SMD:R_0603_1608Metric, symbol Device:R
- removed CN3065_STDBY_LED1: LED, LED_SMD:LED_0805_2012Metric, symbol Device:LED
- removed CN3965_C1: 22uF, Capacitor_SMD:C_0805_2012Metric, symbol Device:C
- removed DIPSW1: Conn_02x05_Odd_Even, Connector:Dip Switch 5pin 1mm SW_DS05-127-2-06BK-SMT-TR, symbol Connector_Generic:Conn_02x05_Odd_Even
- removed DIP_R1: 4k7, Resistor_SMD:R_0603_1608Metric, symbol Device:R
- removed DIP_R2: 1k, Resistor_SMD:R_0603_1608Metric, symbol Device:R
- removed DIP_R3: 20k, Resistor_SMD:R_0603_1608Metric, symbol Device:R
- removed DIP_R4: 200k, Resistor_SMD:R_0603_1608Metric, symbol Device:R
- removed DIP_R5: 2M, Resistor_SMD:R_0603_1608Metric, symbol Device:R
- removed DMP1045U_1: DMP1045U, Package_TO_SOT_SMD:SOT-23, symbol Transistor_FET:DMP1045U
- removed DMP1045_R1, TMPR1: 10K, Resistor_SMD:R_0603_1608Metric, symbol Device:R
- removed DMP1045_SCHOT1: D_Schottky, Diode_SMD:D_1206_3216Metric, symbol Device:D_Schottky
- removed EPS1: ESP32-PSRAM_LY68L6400S, Package_SO:SOIC-8_3.9x4.9mm_P1.27mm, symbol Memory_RAM:ESP32-PSRAM_LY68L6400S
- removed ESP_FLASH2: W25Q128JVS, AeonLabs Storage:WSON8 FLASH SPI SON127P800X600X80-9N, symbol Memory_Flash:SPI_Flash_W25Q128JVS
- removed ExtSW1, ExtSWBAT_PLUG2: Conn_01x03_Female, Connector_JST:JST_SH_SM03B-SRSS-TB_1x03-1MP_P1.00mm_Horizontal, symbol Connector:Conn_01x03_Female
- removed HX1: HX4002, Package_SO:HX4002 SOT95 P280X125-6N, symbol Power_Management:HX4002
- removed HX_C1, HX_C2, HX_C3: 2.2uF, Capacitor_SMD:C_0603_1608Metric, symbol Device:C
- removed I2C_PLUG1: I2C6, Connector_JST:JST_SH_SM04B-SRSS-TB_1x04-1MP_P1.00mm_Horizontal, symbol Connector:Screw_Terminal_01x04
- removed I2C_SCL_R1, I2C_SDA_R1: 10k, Resistor_SMD:R_0603_1608Metric, symbol Device:R
- removed IMU1: LSM6DS3, Sensor_Motion:LSM6DS3 Motion Sensor PQFN50P300X250X86-14N, symbol Sensor_Motion:LSM6DS3
- removed J1: TYPE-C-31-M-12, Connector_USB:USB_C_Receptacle_HRO_TYPE-C-31-M-12, symbol Interface_USB:TYPE-C-31-M-12
- removed LCD1: Conn_01x12_Male, AeonLabs LCDs:1,69 inch LCD IPS TFT, symbol Connector:Conn_01x12_Male
- removed MTRR1: 10k, Resistor_SMD:R_0805_2012Metric, symbol Device:R
- removed MTRT1: NPN, Package_TO_SOT_SMD:SOT-23, symbol MMBT2907A:MMBT2907A
- removed PSR1: 100K, Resistor_SMD:R_0603_1608Metric, symbol Device:R
- removed PWR_PLUG1: Screw_Terminal_01x02, Connector_JST:JST_SH_SM02B-SRSS-TB_1x02-1MP_P1.00mm_Horizontal, symbol Connector:Screw_Terminal_01x02
- removed TP1: VIN, TestPoint:TestPoint_Pad_D1.0mm, symbol Connector:TestPoint
- removed TP2: VOut, TestPoint:TestPoint_Pad_D1.0mm, symbol Connector:TestPoint
- removed TP3: GND, TestPoint:TestPoint_Pad_D1.0mm, symbol Connector:TestPoint
- removed U1: MCP1525-TT, Package_TO_SOT_SMD:SOT-23, symbol Reference_Voltage:MCP1525-TT
- removed U1: ATSHA204A-MAHDA-T, Package_SO:ATSHA204A Auth SOIC8, symbol Device:ATSHA204A-MAHDA-T
- removed U3: Battery_charger_CN3065_QFN8, Package_DFN_QFN:QFN8 3.1x2.9mm QFNn-8 3x3 SON80P400X400X100-9N, symbol Battery_Management:Battery_charger_CN3065_QFN8
- removed U4: AHT20, Sensor_Humidity:AHT20 HT Sensor PSON100P300X300X110-6N, symbol Sensor:AHT20
- removed U6: TEMT6000, Sensor:TEMT6000-SEN, symbol Sensor:TEMT6000
- removed USB_PLUG_R1, USB_PLUG_R3: 5k1, Resistor_SMD:R_0603_1608Metric, symbol Device:R
- removed USB_PLYG_R2: 150K, Resistor_SMD:R_0603_1608Metric, symbol Device:R
Connections:
- no-connect marks 16 -> 7
Other:
- note removed: "1 channel 12Bit ADC with buit in Ohmeter configurable by jumper PIN 1 channel I2C connection"
- note removed: "1uF to 6.8uF"
- note removed: "3V3: R1=47K; R2=15K;"
- note removed: "Authentication & Security"
- note removed: "Battery Charger CN3065"
- note removed: "DC 3V3 step down"
- note removed: "ESP32 Flash Memory"
- note removed: "Luminosity Sensor"
- note removed: "Motion Sensor"
- note removed: "Power Management"
- note removed: "Power Status Sensing"
- note removed: "Power Switch"
- note removed: "Storage and Authentication"
- note removed: "Temperature and Humidity Sensor"
- note removed: "VIN 2.7V to 5.5V"
- note removed: "Vout=0.8x(1+R1/R2)"
- note removed: "onboard sensors"
- note removed: "peripherals"
- title: Smart DAQ Device 1Ch 12Bit ADC / I2C  -> ESP32 S3
- moved on the sheet: ANT1, EC1, EC10, EC11, EC12, EC13, EC14, EC15, EC16, EC17, EC2, EC3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
